File: ergogen/output/pcbs/not_about_money.kicad_pcb (KiCad board)
At the start: 2 copper layers, 118 x 80 mm, 57 parts

Commit message: Update outputs
Parts:
- moved JST1 26.2 mm to (109.5, 70.5)
- moved MH1 19.0 mm to (128.5, 52.5)
- moved PWR1 13.3 mm to (90.3, 71.5)
- moved RST1 9.50 mm to (128.5, 33.8)
- moved MCU1 3.30 mm to (105.3, 42.0)
- moved D1 2.29 mm to (107.1, 98.8)
- moved D10 2.29 mm to (145.1, 79.8)
- moved D11 2.29 mm to (145.1, 60.8)
- moved D12 2.29 mm to (145.1, 41.8)
- moved D13 2.29 mm to (164.1, 98.8)
- moved D14 2.29 mm to (164.1, 79.8)
- moved D15 2.29 mm to (164.1, 60.8)
- moved D16 2.29 mm to (164.1, 41.8)
- moved D17 2.29 mm to (183.1, 98.8)
- moved D18 2.29 mm to (183.1, 79.8)
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Other:
- board text added: "'Not about money' v0.1 by ceoloide"
Changed lines of the file:
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@@
   (footprint "ceoloide:mounting_hole_npth"
     (layer "F.Cu")
-    (at 109.5 52.5 0)
+    (at 128.5 52.5 0)
     (property "Reference" "MH1"
       (at 0 2.55 0)
@@
     (footprint "ceoloide:diode_tht_sod123"
         (layer "B.Cu")
-        (at 107.5 101 90)
+        (at 107.1 98.75 90)
         (property "Reference" "D1"
             (at 0 0 90)
@@
     (footprint "ceoloide:diode_tht_sod123"
         (layer "B.Cu")
-        (at 107.5 82 90)
+        (at 107.1 79.75 90)
         (property "Reference" "D2"
             (at 0 0 90)
@@
     (footprint "ceoloide:diode_tht_sod123"
         (layer "B.Cu")
-        (at 107.5 63 90)
+        (at 107.1 60.75 90)
         (property "Reference" "D3"
             (at 0 0 90)
@@
     (footprint "ceoloide:diode_tht_sod123"
         (layer "B.Cu")
-        (at 107.5 44 90)
+        (at 107.1 41.75 90)
         (property "Reference" "D4"
             (at 0 0 90)
@@
     (footprint "ceoloide:diode_tht_sod123"
         (layer "B.Cu")
-        (at 126.5 101 90)
+        (at 126.1 98.75 90)
         (property "Reference" "D5"
             (at 0 0 90)
@@
     (footprint "ceoloide:diode_tht_sod123"
         (layer "B.Cu")
-        (at 126.5 82 90)
+        (at 126.1 79.75 90)
         (property "Reference" "D6"
             (at 0 0 90)
@@
     (footprint "ceoloide:diode_tht_sod123"
         (layer "B.Cu")
-        (at 126.5 63 90)
+        (at 126.1 60.75 90)
         (property "Reference" "D7"
             (at 0 0 90)
@@
     (footprint "ceoloide:diode_tht_sod123"
         (layer "B.Cu")
-        (at 126.5 44 90)
+        (at 126.1 41.75 90)
         (property "Reference" "D8"
             (at 0 0 90)
@@
     (footprint "ceoloide:diode_tht_sod123"
         (layer "B.Cu")
-        (at 145.5 101 90)
+        (at 145.1 98.75 90)
         (property "Reference" "D9"
             (at 0 0 90)
@@
     (footprint "ceoloide:diode_tht_sod123"
         (layer "B.Cu")
-        (at 145.5 82 90)
+        (at 145.1 79.75 90)
         (property "Reference" "D10"
             (at 0 0 90)
@@
     (footprint "ceoloide:diode_tht_sod123"
         (layer "B.Cu")
-        (at 145.5 63 90)
+        (at 145.1 60.75 90)
         (property "Reference" "D11"
             (at 0 0 90)
@@
     (footprint "ceoloide:diode_tht_sod123"
         (layer "B.Cu")
-        (at 145.5 44 90)
+        (at 145.1 41.75 90)
         (property "Reference" "D12"
             (at 0 0 90)
@@
     (footprint "ceoloide:diode_tht_sod123"
         (layer "B.Cu")
-        (at 164.5 101 90)
+        (at 164.1 98.75 90)
         (property "Reference" "D13"
             (at 0 0 90)
@@
     (footprint "ceoloide:diode_tht_sod123"
         (layer "B.Cu")
-        (at 164.5 82 90)
+        (at 164.1 79.75 90)
         (property "Reference" "D14"
             (at 0 0 90)
@@
     (footprint "ceoloide:diode_tht_sod123"
         (layer "B.Cu")
-        (at 164.5 63 90)
+        (at 164.1 60.75 90)
         (property "Reference" "D15"
             (at 0 0 90)
@@
     (footprint "ceoloide:diode_tht_sod123"
         (layer "B.Cu")
-        (at 164.5 44 90)
+        (at 164.1 41.75 90)
         (property "Reference" "D16"
             (at 0 0 90)
@@
     (footprint "ceoloide:diode_tht_sod123"
         (layer "B.Cu")
-        (at 183.5 101 90)
+        (at 183.1 98.75 90)
         (property "Reference" "D17"
             (at 0 0 90)
@@
     (footprint "ceoloide:diode_tht_sod123"
         (layer "B.Cu")
-        (at 183.5 82 90)
+        (at 183.1 79.75 90)
         (property "Reference" "D18"
             (at 0 0 90)
@@
     (footprint "ceoloide:diode_tht_sod123"
         (layer "B.Cu")
-        (at 183.5 63 90)
+        (at 183.1 60.75 90)
         (property "Reference" "D19"
             (at 0 0 90)
@@
     (footprint "ceoloide:diode_tht_sod123"
         (layer "B.Cu")
-        (at 183.5 44 90)
+        (at 183.1 41.75 90)
         (property "Reference" "D20"
             (at 0 0 90)
@@
     (footprint "ceoloide:diode_tht_sod123"
         (layer "B.Cu")
-        (at 202.5 101 90)
+        (at 202.1 98.75 90)
         (property "Reference" "D21"
             (at 0 0 90)
@@
     (footprint "ceoloide:diode_tht_sod123"
         (layer "B.Cu")
-        (at 202.5 82 90)
+        (at 202.1 79.75 90)
         (property "Reference" "D22"
             (at 0 0 90)
@@
     (footprint "ceoloide:diode_tht_sod123"
         (layer "B.Cu")
-        (at 202.5 63 90)
+        (at 202.1 60.75 90)
         (property "Reference" "D23"
             (at 0 0 90)
@@
     (footprint "ceoloide:diode_tht_sod123"
         (layer "B.Cu")
-        (at 202.5 44 90)
+        (at 202.1 41.75 90)
         (property "Reference" "D24"
             (at 0 0 90)
@@
   (footprint "ceoloide:mcu_nice_nano"
     (layer "B.Cu")
-    (at 102 42 90)
+    (at 105.3 42 90)
     (property "Reference" "MCU1"
       (at 0 -15 90)
@@
   (footprint "ceoloide:power_switch_smd_side"
     (layer "B.Cu")
-    (at 81 62 180)
+    (at 90.3 71.5 180)
     (property "Reference" "PWR1"
       (at -3.6 0 90)
@@
   (footprint "ceoloide:reset_switch_smd_side"
     (layer "B.Cu")
-    (at 119 33.5 0)
+    (at 128.5 33.75 0)
     (property "Reference" "RST1"
       (at 0 0 0)
@@
     (footprint "ceoloide:battery_connector_jst_ph_2"
         (layer "B.Cu")
-        (at 128.5 52.5 90)
+        (at 109.5 70.5 90)
         (property "Reference" "JST1"
             (at 0 4.8 90)
@@
         (thickness 0.15)
       )
-    )
-  )
+      (justify  mirror)
+    )
+  )
+  (gr_text "'Not about money' v0.1 by ceoloide"
+    (at 147.5 67.5 0)
+    (layer "B.SilkS" )
+    (effects
+      (font
+        (size 1 1)
+        (thickness 0.15)
+      )
+      (justify  mirror)
+    )
+  )
