File: ergogen/output/pcbs/not_about_money.kicad_pcb (KiCad board)
At the start: 2 copper layers, 118 x 80 mm, 57 parts

Commit message: Update assets
Connections:
- MCU1 pad 13: P10 -> R2
- MCU1 pad 14: P16 -> R1
- MCU1 pad 8: R1 -> P5
- MCU1 pad 9: R2 -> P6
