File: ergogen/output/pcbs/not_about_money_autorouted.kicad_pcb (KiCad board)
At the start: 2 copper layers, 118 x 80 mm, 57 parts

Commit message: Update assets
Connections:
- MCU1 pad 13: P10 -> R2
- MCU1 pad 14: P16 -> R1
- MCU1 pad 8: R1 -> P5
- MCU1 pad 9: R2 -> P6
Routing:
- net R4: track 0.00 -> 176.2 mm, vias 0 -> 1
- net R3: track 0.00 -> 159.1 mm, vias 0 -> 1
- net R1: track 0.00 -> 142.8 mm, vias 0 -> 2
- net C5: track 0.00 -> 140.4 mm, vias 0 -> 3
- net C6: track 0.00 -> 134.6 mm, vias 0 -> 3
- net R2: track 0.00 -> 129.3 mm, vias 0 -> 2
- net C4: track 0.00 -> 120.7 mm, vias 0 -> 3
- net C1: track 0.00 -> 94.6 mm
- net C3: track 0.00 -> 93.5 mm, vias 0 -> 2
- net C2: track 0.00 -> 85.8 mm, vias 0 -> 1
- net GND: track 0.00 -> 82.0 mm
- net RST: track 0.00 -> 59.2 mm
- net BAT_P: track 0.00 -> 25.6 mm
- net RAW: track 0.00 -> 22.4 mm, vias 0 -> 1
- net c2_r2: track 0.00 -> 2.70 mm
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
Commit message: Update assets
Routing:
- net R1: track 142.8 -> 108.9 mm, vias 2 -> 0
- net C6: track 134.6 -> 161.7 mm, vias 3 -> 4
- net C1: track 94.6 -> 67.6 mm
- net GND: track 82.0 -> 56.2 mm
- net C4: track 120.7 -> 105.5 mm, vias 3 -> 4
- net C5: track 140.4 -> 128.0 mm, vias 3 -> 4
- net C3: track 93.5 -> 103.0 mm, vias 2 -> 3
- net R2: track 129.3 -> 121.7 mm, vias 2 -> 1
- net C2: track 85.8 -> 79.3 mm, vias 1 -> 0
- net R4: track 176.2 -> 182.6 mm
- net BAT_P: track 25.6 -> 19.7 mm, vias 0 -> 1
- net R3: track 159.1 -> 158.5 mm, vias 1 -> 2
- net RAW: track 22.4 -> 23.1 mm

Commit message: Update assets
Routing:
- net C6: track 161.7 -> 135.3 mm, vias 4 -> 3
- net GND: track 56.2 -> 82.0 mm
- net C4: track 105.5 -> 129.6 mm, vias 4 -> 2
- net RST: track 59.2 -> 46.2 mm, vias 0 -> 1
- net R1: track 108.9 -> 121.4 mm, vias 0 -> 2
- net C3: track 103.0 -> 93.9 mm, vias 3 -> 2
- net C5: track 128.0 -> 137.0 mm
- net C2: track 79.3 -> 85.2 mm, vias 0 -> 1
- net BAT_P: track 19.7 -> 25.6 mm, vias 1 -> 0
- net R4: track 182.6 -> 177.7 mm
- net R3: track 158.5 -> 161.0 mm, vias 2 -> 1
- net RAW: track 23.1 -> 22.4 mm
- net C1: track 67.6 -> 67.8 mm, vias 0 -> 2
- net R2: track 121.7 -> 121.6 mm, vias 1 -> 2
