File: ergogen/pcbs/not_about_money_autorouted.kicad_pcb (KiCad board)
At the start: 2 copper layers, 118 x 80 mm, 57 parts

Commit message: Update assets
Parts:
- moved RST1 4.00 mm to (132.5, 33.8)
Routing:
- net C4: track 97.9 -> 119.3 mm
- net R2: track 144.7 -> 164.7 mm, vias 7 -> 5
- net R3: track 178.5 -> 197.3 mm, vias 6 -> 4
- net C6: track 129.3 -> 140.4 mm
- net GND: track 80.8 -> 89.5 mm
- net C2: track 73.2 -> 64.8 mm, vias 0 -> 1
- net R1: track 126.6 -> 133.8 mm
- net C1: track 67.1 -> 72.6 mm, vias 0 -> 1
- net R4: track 185.9 -> 191.1 mm
- net RST: track 45.6 -> 48.8 mm, vias 0 -> 1
- net BAT_P: track 20.0 -> 18.9 mm, vias 1 -> 0
- net C5: track 113.4 -> 112.7 mm
- net c2_r1: track 3.23 -> 2.70 mm
