File: pcbs/not_about_money_autorouted.kicad_pcb (KiCad board)
At the start: 2 copper layers, 118 x 80 mm, 57 parts

Commit message: Update assets
Routing:
- net C1: track 67.8 -> 94.6 mm, vias 2 -> 0
- net C4: track 129.6 -> 106.8 mm, vias 2 -> 3
- net R3: track 161.0 -> 177.7 mm
- net C5: track 137.0 -> 131.9 mm, vias 4 -> 3
- net R1: track 121.4 -> 118.5 mm, vias 2 -> 1
- net C6: track 135.3 -> 133.2 mm, vias 3 -> 2
- net C3: track 93.9 -> 95.5 mm
- net R2: track 121.6 -> 122.4 mm
- net R4: track 177.7 -> 177.0 mm
- net C2: track 85.2 -> 85.8 mm

Commit message: Update assets
Routing:
- net R3: track 177.7 -> 155.3 mm, vias 1 -> 2
- net C2: track 85.8 -> 74.3 mm
- net R1: track 118.5 -> 113.9 mm
- net C3: track 95.5 -> 99.3 mm, vias 2 -> 3
- net C5: track 131.9 -> 133.8 mm, vias 3 -> 4
- net C4: track 106.8 -> 108.4 mm, vias 3 -> 4
- net RST: track 46.2 -> 44.8 mm, vias 1 -> 0
- net C6: track 133.2 -> 134.6 mm, vias 2 -> 3
- net R2: track 122.4 -> 121.2 mm, vias 2 -> 1
- net RAW: track 22.4 -> 23.6 mm
- net R4: track 177.0 -> 176.0 mm
- net BAT_P: track 25.6 -> 24.7 mm
- net c6_r2: track 2.70 -> 3.23 mm
- net c6_r1: track 2.70 -> 3.23 mm
- net c5_r2: track 2.70 -> 3.23 mm
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